Commit message: Change support polygon with Start + Fix desired 3D acceleration

File: bauzil_stairs.urdf (robot description, URDF)
Before this commit: robot bauzil_stairs.urdf, 1 links, 0 joints
Links:
- link baseLink: geometry collision mesh filename=bauzil_stairs.stl scale=1.3 1.3 0.2; visual mesh filename=bauzil_stairs.stl scale=1.3 1.3 0.2

Commit message: Rescale bauzil stairs

File: bauzil_stairs.urdf (robot description, URDF)
Before this commit: robot bauzil_stairs.urdf, 1 links, 0 joints
Links:
- link baseLink: geometry collision mesh filename=bauzil_stairs.stl scale=0.7 1.0 0.5; visual mesh filename=bauzil_stairs.stl scale=0.7 1.0 0.5
